Commit message: Measured geometry 2026-08-05: hanging bench, planar arms, calibrated URDF
The caliper session replaced every estimated arm dimension and revealed
the real bench configuration, which the model now follows:

- dimensions.yaml: every arm-chain length measured on the right arm,
  new bench section (central box, plate, column anchors), provenance
  per entry. Manual-photo estimates were off by up to 40 mm (upper arm
  79.3 mm real vs 120 estimated).
- soma_arm.xacro: the arm as built, not as the manual drew it. Both
  arms HANG from their slew discs; J1 to J4 axes are PARALLEL (each arm
  a planar 4R chain plus wrist roll), with a 33 mm clavicle link from
  disc center to shoulder axis. New `side` parameter mirrors the
  hug-convention joint sense between arms. Axis signs stay provisional
  until the first powered RViz-vs-reality check (v0.2).
- soma_bench.urdf.xacro: the real rig as one static bench link (plate,
  column, central box) with both arms hanging. FK cross-check: at zero
  the fingertips sit 5.7 mm above the plate, matching the photos.
- Torso: dormant design (no L16 on this bench). The sync script
  tolerates exactly that joint off-model; ros2_control layer and
  controllers.yaml park their lift entries with the same note.
- smoke_test.sh: end to end is now a left elbow bend to its soft limit;
  TF must confirm the measured 225 mm tool lift.
- Suite: 85 passed + 1 skipped; model-driver sync green on the expanded
  bench URDF.

Co-Authored-By: Claude Fable 5 <noreply@anthropic.com>

File: soma_description/urdf/single_arm.urdf.xacro (robot description, xacro)
@@ -1,6 +1,8 @@
 <?xml version="1.0"?>
 <!--
-  One 6DOF arm bolted to the bench, for studying and calibrating a single
-  arm in isolation. This is the model to use with calipers in hand.
+  One 6DOF arm hanging in isolation, for studying and calibrating a
+  single arm. Mounted exactly like the RIGHT arm on the bench (same
+  height, same orientation, same side=-1 hug sense), minus the bench
+  geometry, so numbers read here transfer 1:1 to the full model.
   Usage:
     ros2 launch soma_description display.launch.py model:=single_arm.urdf.xacro
@@ -10,6 +12,6 @@
   <xacro:include filename="$(find soma_description)/urdf/soma_arm.xacro"/>
   <link name="world"/>
-  <xacro:soma_arm prefix="arm_" parent="world">
-    <origin xyz="0 0 0" rpy="0 0 0"/>
+  <xacro:soma_arm prefix="arm_" parent="world" side="-1">
+    <origin xyz="0 0 0.343" rpy="${pi/2} ${pi/2} 0"/>
   </xacro:soma_arm>
 </robot>

File: soma_description/urdf/soma_arm.xacro (robot description, xacro)
@@ -4,43 +4,53 @@
   Hardware: "6DOF metal robot arm" sold by ThanksBuyer / Red Sun Global
   (AliExpress item 1005007215923987), bought as the "Arm Only" variant and
-  fitted with our own MG996R servos. The kit ships a 30 page assembly
-  manual; page 28 labels the six joints A to F on the physical arm, and
-  that labelling is the source of the chain below. Full part numbers and
-  datasheets: docs/hardware.md.
-  Chain, exactly as the manual labels it:
-    A = base yaw (on the large slew bearing)  -> ${prefix}yaw_joint         (Z)
-    B = shoulder pitch                        -> ${prefix}shoulder_joint    (Y)
-    C = elbow pitch (twin servo block)        -> ${prefix}elbow_joint       (Y)
-    D = wrist pitch                           -> ${prefix}wrist_pitch_joint (Y)
-    E = wrist roll                            -> ${prefix}wrist_roll_joint  (local Z)
-    F = geared two finger gripper             -> ${prefix}finger_l_joint + mimic
-  Servos: 40x20 body, 25T spline. The frame is designed for 25 kg.cm class
-  servos; we fit MG996R (about 10 kg.cm), so shoulder and base are the
-  joints to watch under load. Swapping just those two for a stronger servo
-  is a non destructive upgrade.
-  EVERY length below is marked [calibrate]: they are estimated from the
-  manual photos and from the standard dimensions of this frame family.
-  They get measured with calipers and corrected here ONCE, and the whole
-  model follows. This is the deliverable of v0.1.
-  Modelled in the "candle" pose (arm pointing along +Z, every joint at
-  zero). REP-103 convention. Roughly 0.9 kg per arm with six servos.
+  fitted with our own MG996R servos. The kit manual labels the joints A to
+  F; the joint NAMES below keep that lineage (they are also the driver's
+  channel labels in servo_map.py, so they never change lightly).
+  MEASURED TRUTH, 2026-08-05 caliper session. The arm as actually built
+  and mounted is NOT the manual's upright yaw-first chain:
+    - The arm HANGS from its slew disc. The disc axis (J1) is HORIZONTAL,
+      pointing outboard. J1 swings the whole arm forward/backward like a
+      pendulum.
+    - J1, J2 (shoulder), J3 (elbow) and J4 (wrist pitch) axes are ALL
+      PARALLEL: the arm is a planar 4R chain in its own vertical plane,
+      redundant like a finger. J5 (wrist roll) spins the gripper about
+      the forearm axis and is what moves the fingertips out of plane.
+    - A 33 mm link Andres named "the clavicle" joins the disc center to
+      the shoulder axis.
+  Local frame of the macro root (${prefix}mount_link), chosen so one rpy
+  at the mount does all the work:
+    +Z  along the disc axis, pointing OUTBOARD (away from the bench box)
+    +X  the chain direction at zero pose (world DOWN once mounted)
+  Mount with rpy such that +X maps to world -Z; see soma_bench.urdf.xacro.
+  The `side` parameter mirrors the joint SENSE, not the geometry: the hug
+  convention (negative = inward, closing a hug; positive = outward/up) is
+  mirror-symmetric between arms by definition, so the left arm uses
+  side=1 and the right arm side=-1 on every revolute axis.
+  AXIS SIGNS ARE PROVISIONAL: lengths, parallelism and anchors are
+  caliper-measured; the world-direction of each joint's positive sense
+  still needs the first powered RViz-vs-reality comparison (v0.2 session,
+  one small commanded angle per joint). A wrong sense is a one-line flip
+  here plus the same flip in the mirror. Do not "fix" signs from the
+  armchair; fix them from the bench.
+  Visuals are honest bounding boxes; pretty geometry arrives with the
+  CAD-to-URDF pipeline (task #30). Roughly 0.7 kg per hanging arm (the
+  base boxes now live in the bench model).
 -->
 <robot xmlns:xacro="http://www.ros.org/wiki/xacro">
-  <!-- ==================== dimensions [calibrate] ==================== -->
-  <xacro:property name="base_lx"        value="0.095"/>  <!-- base box, houses servo A -->
-  <xacro:property name="base_ly"        value="0.095"/>
-  <xacro:property name="base_lz"        value="0.062"/>
-  <xacro:property name="turntable_r"    value="0.042"/>  <!-- disc on the slew bearing -->
-  <xacro:property name="turntable_h"    value="0.012"/>
-  <xacro:property name="shoulder_off_z" value="0.045"/>  <!-- disc to shoulder axis -->
-  <xacro:property name="upper_len"      value="0.120"/>  <!-- shoulder to elbow -->
-  <xacro:property name="fore_len"       value="0.090"/>  <!-- elbow to wrist pitch -->
-  <xacro:property name="wrist_len"      value="0.055"/>  <!-- wrist pitch to roll flange -->
-  <xacro:property name="gripper_base_h" value="0.045"/>  <!-- roll flange to finger axis -->
-  <xacro:property name="finger_len"     value="0.075"/>  <!-- geared finger -->
-  <xacro:property name="finger_sep"     value="0.024"/>  <!-- gear axis separation -->
-  <xacro:property name="plate_w"        value="0.030"/>  <!-- link plate width -->
-  <xacro:property name="plate_t"        value="0.060"/>  <!-- plate pair depth -->
-  <!-- MG996R class servo, 40x20 body -->
+  <!-- ============ dimensions, MEASURED 2026-08-05 ============
+       Every literal here has a provenance row in config/dimensions.yaml;
+       test_dimensions_sync.py keeps the two in agreement. -->
+  <xacro:property name="disc_r"         value="0.02455"/> <!-- slew disc, the one that rotates -->
+  <xacro:property name="disc_h"         value="0.0074"/>  <!-- disc protrusion from its box -->
+  <xacro:property name="clavicle_len"   value="0.033"/>   <!-- disc center to shoulder axis -->
+  <xacro:property name="upper_len"      value="0.0793"/>  <!-- shoulder to elbow -->
+  <xacro:property name="fore_len"       value="0.075"/>   <!-- elbow to wrist pitch -->
+  <xacro:property name="wrist_len"      value="0.0664"/>  <!-- wrist pitch to gripper mount face -->
+  <xacro:property name="gripper_base_h" value="0.0179"/>  <!-- mount face to finger gear axes -->
+  <xacro:property name="finger_len"     value="0.0657"/>  <!-- gear axis to fingertip -->
+  <xacro:property name="finger_sep"     value="0.0257"/>  <!-- between the two gear axes -->
+  <xacro:property name="plate_w"        value="0.0319"/>  <!-- link plate width -->
+  <xacro:property name="plate_t"        value="0.0528"/>  <!-- arm sandwich outer width -->
+  <!-- MG996R class servo, 40x20 body (datasheet) -->
   <xacro:property name="servo_lx" value="0.041"/>
   <xacro:property name="servo_ly" value="0.020"/>
@@ -51,5 +61,5 @@
        were closing a hug, grasping features facing forward; positive =
        outward/up. Limits are asymmetric and differ per side, so they are
-       macro parameters below (defaults = RIGHT arm; the torso passes the
+       macro parameters below (defaults = RIGHT arm; the bench passes the
        left values). They MUST stay in sync with SERVO_MAP in
        soma_driver/servo_map.py; CI checks exactly that. -->
@@ -71,15 +81,7 @@
     </inertial>
   </xacro:macro>
-  <!-- visual of a 40x20 servo (red box) -->
-  <xacro:macro name="servo_visual" params="xyz rpy:='0 0 0'">
-    <visual>
-      <origin xyz="${xyz}" rpy="${rpy}"/>
-      <geometry><box size="${servo_lx} ${servo_ly} ${servo_lz}"/></geometry>
-      <material name="servo_red"/>
-    </visual>
-  </xacro:macro>
   <!-- ==================== the arm macro ==================== -->
   <xacro:macro name="soma_arm"
-               params="prefix parent *origin
+               params="prefix parent side:=1 *origin
                        yaw_lower:=-2.7960 yaw_upper:=0.3456
                        shoulder_lower:=-0.4712 shoulder_upper:=2.3562
@@ -87,130 +89,116 @@
                        wrist_pitch_lower:=-2.0420 wrist_pitch_upper:=0.8482
                        wrist_roll_lower:=-1.8222 wrist_roll_upper:=1.2724">
-    <!-- mount to the parent link -->
+    <!-- mount to the parent link, at the disc seat on the bench box -->
     <joint name="${prefix}mount_joint" type="fixed">
       <parent link="${parent}"/>
-      <child link="${prefix}base_link"/>
+      <child link="${prefix}mount_link"/>
       <xacro:insert_block name="origin"/>
     </joint>
-    <!-- base: metal box holding servo A and the wiring -->
-    <link name="${prefix}base_link">
-      <visual>
-        <origin xyz="0 0 ${base_lz/2}"/>
-        <geometry><box size="${base_lx} ${base_ly} ${base_lz}"/></geometry>
-        <material name="aluminum"/>
-      </visual>
-      <collision>
-        <origin xyz="0 0 ${base_lz/2}"/>
-        <geometry><box size="${base_lx} ${base_ly} ${base_lz}"/></geometry>
-      </collision>
-      <xacro:box_inertia m="0.25" x="${base_lx}" y="${base_ly}" z="${base_lz}"/>
-    </link>
-    <!-- A: base yaw on the slew bearing -->
+    <link name="${prefix}mount_link"/>
+    <!-- A: the slew disc, J1. Horizontal axis, the arm's fore/aft swing. -->
     <joint name="${prefix}yaw_joint" type="revolute">
-      <parent link="${prefix}base_link"/>
+      <parent link="${prefix}mount_link"/>
       <child link="${prefix}turntable_link"/>
-      <origin xyz="0 0 ${base_lz}"/>
-      <axis xyz="0 0 1"/>
+      <origin xyz="0 0 0"/>
+      <axis xyz="0 0 ${side}"/>
       <limit lower="${yaw_lower}" upper="${yaw_upper}" effort="${effort_nm}" velocity="${vel_rads}"/>
     </joint>
+    <!-- disc plus the clavicle bracket that carries the shoulder servo -->
     <link name="${prefix}turntable_link">
       <visual>
-        <origin xyz="0 0 ${turntable_h/2}"/>
-        <geometry><cylinder radius="${turntable_r}" length="${turntable_h}"/></geometry>
+        <origin xyz="0 0 ${disc_h/2}"/>
+        <geometry><cylinder radius="${disc_r}" length="${disc_h}"/></geometry>
         <material name="dark_gray"/>
       </visual>
-      <!-- shoulder yoke -->
-      <visual>
-        <origin xyz="0 0 ${turntable_h + shoulder_off_z/2}"/>
-        <geometry><box size="0.050 0.070 ${shoulder_off_z}"/></geometry>
-        <material name="aluminum"/>
-      </visual>
-      <collision>
-        <origin xyz="0 0 ${(turntable_h + shoulder_off_z)/2}"/>
-        <geometry><box size="0.070 0.080 ${turntable_h + shoulder_off_z}"/></geometry>
-      </collision>
-      <xacro:box_inertia m="0.12" x="0.07" y="0.08" z="${turntable_h + shoulder_off_z}"/>
-    </link>
-    <!-- B: shoulder -->
+      <visual>
+        <origin xyz="${clavicle_len/2} 0 ${disc_h + 0.003}"/>
+        <geometry><box size="${clavicle_len + 0.030} 0.030 0.006"/></geometry>
+        <material name="aluminum"/>
+      </visual>
+      <collision>
+        <origin xyz="${clavicle_len/2} 0 ${disc_h/2 + 0.003}"/>
+        <geometry><box size="${clavicle_len + 2*disc_r} 0.050 ${disc_h + 0.006}"/></geometry>
+      </collision>
+      <xacro:box_inertia m="0.10" x="${clavicle_len + 2*disc_r}" y="0.05" z="${disc_h + 0.006}"/>
+    </link>
+    <!-- B: shoulder. PARALLEL to J1, one clavicle away. -->
     <joint name="${prefix}shoulder_joint" type="revolute">
       <parent link="${prefix}turntable_link"/>
       <child link="${prefix}upper_arm_link"/>
-      <origin xyz="0 0 ${turntable_h + shoulder_off_z}"/>
-      <axis xyz="0 1 0"/>
+      <origin xyz="${clavicle_len} 0 ${disc_h}"/>
+      <axis xyz="0 0 ${side}"/>
       <limit lower="${shoulder_lower}" upper="${shoulder_upper}" effort="${effort_nm}" velocity="${vel_rads}"/>
     </joint>
     <link name="${prefix}upper_arm_link">
       <visual>
-        <origin xyz="0 0 ${upper_len/2}"/>
-        <geometry><box size="${plate_w} ${plate_t} ${upper_len}"/></geometry>
-        <material name="aluminum"/>
-      </visual>
-      <xacro:servo_visual xyz="0 ${plate_t/2 + servo_ly/2} 0"/>
-      <collision>
-        <origin xyz="0 0 ${upper_len/2}"/>
-        <geometry><box size="${plate_w} ${plate_t + 2*servo_ly} ${upper_len}"/></geometry>
-      </collision>
-      <xacro:box_inertia m="0.18" x="${plate_w}" y="${plate_t}" z="${upper_len}"/>
-    </link>
-    <!-- C: elbow (twin servo block, manual page 15) -->
+        <origin xyz="${upper_len/2} 0 0"/>
+        <geometry><box size="${upper_len} ${plate_w} ${plate_t}"/></geometry>
+        <material name="aluminum"/>
+      </visual>
+      <collision>
+        <origin xyz="${upper_len/2} 0 0"/>
+        <geometry><box size="${upper_len + 0.02} ${plate_w + 0.01} ${plate_t + 0.01}"/></geometry>
+      </collision>
+      <xacro:box_inertia m="0.18" x="${upper_len}" y="${plate_w}" z="${plate_t}"/>
+    </link>
+    <!-- C: elbow (twin servo block). Parallel again. -->
     <joint name="${prefix}elbow_joint" type="revolute">
       <parent link="${prefix}upper_arm_link"/>
       <child link="${prefix}forearm_link"/>
-      <origin xyz="0 0 ${upper_len}"/>
-      <axis xyz="0 1 0"/>
+      <origin xyz="${upper_len} 0 0"/>
+      <axis xyz="0 0 ${side}"/>
       <limit lower="${elbow_lower}" upper="${elbow_upper}" effort="${effort_nm}" velocity="${vel_rads}"/>
     </joint>
     <link name="${prefix}forearm_link">
       <visual>
-        <origin xyz="0 0 ${fore_len/2}"/>
-        <geometry><box size="${plate_w} ${plate_t} ${fore_len}"/></geometry>
-        <material name="aluminum"/>
-      </visual>
-      <xacro:servo_visual xyz="0 ${-(plate_t/2 + servo_ly/2)} 0"/>
-      <collision>
-        <origin xyz="0 0 ${fore_len/2}"/>
-        <geometry><box size="${plate_w} ${plate_t + 2*servo_ly} ${fore_len}"/></geometry>
-      </collision>
-      <xacro:box_inertia m="0.16" x="${plate_w}" y="${plate_t}" z="${fore_len}"/>
-    </link>
-    <!-- D: wrist pitch -->
+        <origin xyz="${fore_len/2} 0 0"/>
+        <geometry><box size="${fore_len} ${plate_w} ${plate_t}"/></geometry>
+        <material name="aluminum"/>
+      </visual>
+      <collision>
+        <origin xyz="${fore_len/2} 0 0"/>
+        <geometry><box size="${fore_len + 0.02} ${plate_w + 0.01} ${plate_t + 0.01}"/></geometry>
+      </collision>
+      <xacro:box_inertia m="0.16" x="${fore_len}" y="${plate_w}" z="${plate_t}"/>
+    </link>
+    <!-- D: wrist pitch. Last of the parallel four. -->
     <joint name="${prefix}wrist_pitch_joint" type="revolute">
       <parent link="${prefix}forearm_link"/>
       <child link="${prefix}wrist_link"/>
-      <origin xyz="0 0 ${fore_len}"/>
-      <axis xyz="0 1 0"/>
+      <origin xyz="${fore_len} 0 0"/>
+      <axis xyz="0 0 ${side}"/>
       <limit lower="${wrist_pitch_lower}" upper="${wrist_pitch_upper}" effort="${effort_nm}" velocity="${vel_rads}"/>
     </joint>
     <link name="${prefix}wrist_link">
       <visual>
-        <origin xyz="0 0 ${wrist_len/2}"/>
-        <geometry><box size="0.040 0.045 ${wrist_len}"/></geometry>
-        <material name="aluminum"/>
-      </visual>
-      <collision>
-        <origin xyz="0 0 ${wrist_len/2}"/>
-        <geometry><box size="0.045 0.050 ${wrist_len}"/></geometry>
-      </collision>
-      <xacro:box_inertia m="0.09" x="0.04" y="0.045" z="${wrist_len}"/>
-    </link>
-    <!-- E: wrist roll (spins the gripper about the arm axis) -->
+        <origin xyz="${wrist_len/2} 0 0"/>
+        <geometry><box size="${wrist_len} 0.040 0.045"/></geometry>
+        <material name="aluminum"/>
+      </visual>
+      <collision>
+        <origin xyz="${wrist_len/2} 0 0"/>
+        <geometry><box size="${wrist_len} 0.045 0.050"/></geometry>
+      </collision>
+      <xacro:box_inertia m="0.09" x="${wrist_len}" y="0.04" z="0.045"/>
+    </link>
+    <!-- E: wrist roll, about the forearm axis. The out-of-plane joint. -->
     <joint name="${prefix}wrist_roll_joint" type="revolute">
       <parent link="${prefix}wrist_link"/>
       <child link="${prefix}gripper_base_link"/>
-      <origin xyz="0 0 ${wrist_len}"/>
-      <axis xyz="0 0 1"/>
+      <origin xyz="${wrist_len} 0 0"/>
+      <axis xyz="${side} 0 0"/>
       <limit lower="${wrist_roll_lower}" upper="${wrist_roll_upper}" effort="${effort_nm}" velocity="${vel_rads}"/>
     </joint>
     <link name="${prefix}gripper_base_link">
       <visual>
-        <origin xyz="0 0 ${gripper_base_h/2}"/>
-        <geometry><box size="0.045 0.038 ${gripper_base_h}"/></geometry>
+        <origin xyz="${gripper_base_h/2} 0 0"/>
+        <geometry><box size="${gripper_base_h} 0.038 0.045"/></geometry>
         <material name="dark_gray"/>
       </visual>
       <collision>
-        <origin xyz="0 0 ${gripper_base_h/2}"/>
-        <geometry><box size="0.045 0.038 ${gripper_base_h}"/></geometry>
-      </collision>
-      <xacro:box_inertia m="0.10" x="0.045" y="0.038" z="${gripper_base_h}"/>
+        <origin xyz="${gripper_base_h/2} 0 0"/>
+        <geometry><box size="${gripper_base_h} 0.038 0.045"/></geometry>
+      </collision>
+      <xacro:box_inertia m="0.12" x="${gripper_base_h}" y="0.038" z="0.045"/>
     </link>
     <!-- F: geared gripper. Left finger is driven, right one mirrors it. -->
@@ -218,25 +206,25 @@
       <parent link="${prefix}gripper_base_link"/>
       <child link="${prefix}finger_l_link"/>
-      <origin xyz="0 ${finger_sep/2} ${gripper_base_h}"/>
-      <axis xyz="1 0 0"/>
+      <origin xyz="${gripper_base_h} 0 ${finger_sep/2}"/>
+      <axis xyz="0 1 0"/>
       <limit lower="0.0" upper="1.0" effort="${effort_nm}" velocity="${vel_rads}"/>
     </joint>
     <link name="${prefix}finger_l_link">
       <visual>
-        <origin xyz="0 0.004 ${finger_len/2}"/>
-        <geometry><box size="0.010 0.008 ${finger_len}"/></geometry>
-        <material name="aluminum"/>
-      </visual>
-      <collision>
-        <origin xyz="0 0.004 ${finger_len/2}"/>
-        <geometry><box size="0.010 0.008 ${finger_len}"/></geometry>
-      </collision>
-      <xacro:box_inertia m="0.02" x="0.01" y="0.008" z="${finger_len}"/>
+        <origin xyz="${finger_len/2} 0 0.004"/>
+        <geometry><box size="${finger_len} 0.010 0.008"/></geometry>
+        <material name="aluminum"/>
+      </visual>
+      <collision>
+        <origin xyz="${finger_len/2} 0 0.004"/>
+        <geometry><box size="${finger_len} 0.010 0.008"/></geometry>
+      </collision>
+      <xacro:box_inertia m="0.03" x="${finger_len}" y="0.01" z="0.008"/>
     </link>
     <joint name="${prefix}finger_r_joint" type="revolute">
       <parent link="${prefix}gripper_base_link"/>
       <child link="${prefix}finger_r_link"/>
-      <origin xyz="0 ${-finger_sep/2} ${gripper_base_h}"/>
-      <axis xyz="1 0 0"/>
+      <origin xyz="${gripper_base_h} 0 ${-finger_sep/2}"/>
+      <axis xyz="0 1 0"/>
       <limit lower="-1.0" upper="0.0" effort="${effort_nm}" velocity="${vel_rads}"/>
       <mimic joint="${prefix}finger_l_joint" multiplier="-1.0"/>
@@ -244,13 +232,13 @@
     <link name="${prefix}finger_r_link">
       <visual>
-        <origin xyz="0 -0.004 ${finger_len/2}"/>
-        <geometry><box size="0.010 0.008 ${finger_len}"/></geometry>
-        <material name="aluminum"/>
-      </visual>
-      <collision>
-        <origin xyz="0 -0.004 ${finger_len/2}"/>
-        <geometry><box size="0.010 0.008 ${finger_len}"/></geometry>
-      </collision>
-      <xacro:box_inertia m="0.02" x="0.01" y="0.008" z="${finger_len}"/>
+        <origin xyz="${finger_len/2} 0 -0.004"/>
+        <geometry><box size="${finger_len} 0.010 0.008"/></geometry>
+        <material name="aluminum"/>
+      </visual>
+      <collision>
+        <origin xyz="${finger_len/2} 0 -0.004"/>
+        <geometry><box size="${finger_len} 0.010 0.008"/></geometry>
+      </collision>
+      <xacro:box_inertia m="0.03" x="${finger_len}" y="0.01" z="0.008"/>
     </link>
     <!-- tool frame (gripper tip, the IK target for MoveIt2) -->
@@ -258,5 +246,5 @@
       <parent link="${prefix}gripper_base_link"/>
       <child link="${prefix}tool0"/>
-      <origin xyz="0 0 ${gripper_base_h + finger_len}"/>
+      <origin xyz="${gripper_base_h + finger_len} 0 0"/>
     </joint>
     <link name="${prefix}tool0"/>
