Commit message: The measured map: re-splined zeros, asymmetric limits, the hug convention
On 2026-08-03 every horn was re-splined with its servo holding the
electrical center, and the mechanical zero plus both travel limits were
captured per channel with the workbench. This commit makes that capture
the law of the repo:

- SERVO_MAP now carries the measured rows. Sign convention (the hug
  rule): negative = inward, as if closing a hug, grasping features
  forward; positive = outward/up. Four arm channels are inverted
  (min_us > max_us) because that is how the mirrored geometry measures:
  rolls and yaws invert on opposite arms, elbows on both.
- The xacro grows per-joint limit parameters (defaults = right arm, the
  torso passes the left arm's), so the URDF carries the same asymmetric
  truth and CI keeps both in sync.
- Tests that pinned the old assumed map (symmetric 90 deg around 1500 us)
  are rewritten to pin the measured one, explicitly allowed because the
  hardware fact changed. 82 pass, 1 skipped.
- Raw capture versioned at calibration/servo_calibration_2026-08-03.json.

Known flags, encoded rather than hidden: left yaw's zero sits AT its
2500 us stop (upper = 0.0, re-spline one tooth pending, there is a test
that will demand updating when it happens) and the grippers open
different amounts (1490 vs 1030 us, physical check pending).

Co-Authored-By: Claude Fable 5 <noreply@anthropic.com>

File: soma_description/urdf/soma_arm.xacro (robot description, xacro)
@@ -46,7 +46,12 @@
   <xacro:property name="servo_ly" value="0.020"/>
   <xacro:property name="servo_lz" value="0.038"/>
-  <!-- Limits: 180 degree servos, so +/- 90 from center. These MUST stay in
-       sync with SERVO_MAP in soma_driver/servo_map.py. -->
-  <xacro:property name="lim"        value="${pi/2}"/>
+  <!-- Limits: MEASURED on 2026-08-03, joint by joint, after re-splining
+       every horn so the mechanical zero matches the electrical center.
+       Convention (Andres's "hug rule"): negative = inward, as if the robot
+       were closing a hug, grasping features facing forward; positive =
+       outward/up. Limits are asymmetric and differ per side, so they are
+       macro parameters below (defaults = RIGHT arm; the torso passes the
+       left values). They MUST stay in sync with SERVO_MAP in
+       soma_driver/servo_map.py; CI checks exactly that. -->
   <xacro:property name="effort_nm"  value="1.0"/>   <!-- MG996R ~10 kg.cm = 0.98 N.m -->
   <xacro:property name="vel_rads"   value="3.0"/>   <!-- ~0.17 s/60 deg plus margin -->
@@ -75,5 +80,11 @@
   </xacro:macro>
   <!-- ==================== the arm macro ==================== -->
-  <xacro:macro name="soma_arm" params="prefix parent *origin">
+  <xacro:macro name="soma_arm"
+               params="prefix parent *origin
+                       yaw_lower:=-2.7960 yaw_upper:=0.3456
+                       shoulder_lower:=-0.4712 shoulder_upper:=2.3562
+                       elbow_lower:=-2.1363 elbow_upper:=0.9739
+                       wrist_pitch_lower:=-2.0420 wrist_pitch_upper:=0.8482
+                       wrist_roll_lower:=-1.8222 wrist_roll_upper:=1.2724">
     <!-- mount to the parent link -->
     <joint name="${prefix}mount_joint" type="fixed">
@@ -101,5 +112,5 @@
       <origin xyz="0 0 ${base_lz}"/>
       <axis xyz="0 0 1"/>
-      <limit lower="${-lim}" upper="${lim}" effort="${effort_nm}" velocity="${vel_rads}"/>
+      <limit lower="${yaw_lower}" upper="${yaw_upper}" effort="${effort_nm}" velocity="${vel_rads}"/>
     </joint>
     <link name="${prefix}turntable_link">
@@ -127,5 +138,5 @@
       <origin xyz="0 0 ${turntable_h + shoulder_off_z}"/>
       <axis xyz="0 1 0"/>
-      <limit lower="${-lim}" upper="${lim}" effort="${effort_nm}" velocity="${vel_rads}"/>
+      <limit lower="${shoulder_lower}" upper="${shoulder_upper}" effort="${effort_nm}" velocity="${vel_rads}"/>
     </joint>
     <link name="${prefix}upper_arm_link">
@@ -148,5 +159,5 @@
       <origin xyz="0 0 ${upper_len}"/>
       <axis xyz="0 1 0"/>
-      <limit lower="${-lim}" upper="${lim}" effort="${effort_nm}" velocity="${vel_rads}"/>
+      <limit lower="${elbow_lower}" upper="${elbow_upper}" effort="${effort_nm}" velocity="${vel_rads}"/>
     </joint>
     <link name="${prefix}forearm_link">
@@ -169,5 +180,5 @@
       <origin xyz="0 0 ${fore_len}"/>
       <axis xyz="0 1 0"/>
-      <limit lower="${-lim}" upper="${lim}" effort="${effort_nm}" velocity="${vel_rads}"/>
+      <limit lower="${wrist_pitch_lower}" upper="${wrist_pitch_upper}" effort="${effort_nm}" velocity="${vel_rads}"/>
     </joint>
     <link name="${prefix}wrist_link">
@@ -189,5 +200,5 @@
       <origin xyz="0 0 ${wrist_len}"/>
       <axis xyz="0 0 1"/>
-      <limit lower="${-lim}" upper="${lim}" effort="${effort_nm}" velocity="${vel_rads}"/>
+      <limit lower="${wrist_roll_lower}" upper="${wrist_roll_upper}" effort="${effort_nm}" velocity="${vel_rads}"/>
     </joint>
     <link name="${prefix}gripper_base_link">

File: soma_description/urdf/soma_torso.xacro (robot description, xacro)
@@ -133,6 +133,13 @@
       </inertial>
     </link>
-    <!-- the two arms, splayed at +/- 45 deg -->
-    <xacro:soma_arm prefix="left_arm_" parent="torso_plate_link">
+    <!-- the two arms, splayed at +/- 45 deg. Joint limits were MEASURED
+         per side on 2026-08-03 (hug convention: negative = inward); the
+         macro defaults carry the right arm, the left passes its own. -->
+    <xacro:soma_arm prefix="left_arm_" parent="torso_plate_link"
+                    yaw_lower="-3.0788" yaw_upper="0.0"
+                    shoulder_lower="-0.3927" shoulder_upper="2.1206"
+                    elbow_lower="-1.5708" elbow_upper="0.7854"
+                    wrist_pitch_lower="-1.6179" wrist_pitch_upper="1.0996"
+                    wrist_roll_lower="-1.5080" wrist_roll_upper="1.3509">
       <origin xyz="${arm_x} ${arm_y} ${plate_lz}" rpy="0 0 ${arm_yaw}"/>
     </xacro:soma_arm>

Commit message: Jetson operating docs: gate 1 by relaunch, what arming really sends, the ATX stop
docker-compose.jetson.yml launches with allow_real:=${ALLOW_REAL:-false},
so gate 1 finally has a recipe on the Jetson: ALLOW_REAL=true ... up -d
--force-recreate, closed again by a plain relaunch. The header names
two traps: restart: unless-stopped keeps a container's configuration
across reboots (one created with ALLOW_REAL=true comes back with gate 1
open), and compose reads .env on its own (ALLOW_REAL never goes there).
`docker compose config` validates both forms.

docs/bench.md, new section 6: ssh, i2cdetect on bus 7, compose up /
logs / down, how new code reaches the driver, a `soma` helper that
passes arguments as positional parameters (splicing $* into bash -c
splits "{data: true}" in two), a self-test of its quoting, and a "can
it move a motor" table.

docs/safety.md: the Jetson commands for both gates; and a correction.
The page said the arming call never causes motion. It does: the next
tick sends every channel the pulse of the pose the driver believes it
holds, at once, and the ramp cannot shape that move because the driver
believes the joint is already there. Hanging gravity joints sit near
zero; wrist rolls and grippers can snap. TestWhatArmingSends (ROS job)
pins both cases, including a believed pose that is not zero. Rule 4 now
names its two blind moments. The emergency stop is the ATX rear switch;
pulling the XT60 under load is not a stop.

docs/wiring.md: today's power chain (ATX, 10 A fuse, XT60, Y splitter,
one 6 V UBEC per board, the Jetson on its own adapter, INA3221 off the
bus), bus 7 with 0x40 and 0x43, and the Jetson bring-up order,
including silencing both boards (ALL_LED_OFF_H full off, the write
disable_all() makes) before V+ comes up.

docs/plan.md, docs/log.md (dated clarification), the soma_arm.xacro
comment and the workspace_map.py docstring: metal reversed is a driver
fix (mirror the SERVO_MAP row) and the reach map is then rerun WITHOUT
--flip; RViz reversed with the metal right is an axis flip, which the
map never reads. --flip is only a preview before a driver fix lands.
README: the emergency stop is the switch that feeds the servo rail.

Co-Authored-By: Claude Opus 5.5 <noreply@anthropic.com>

File: soma_description/urdf/soma_arm.xacro (robot description, xacro)
@@ -29,8 +29,13 @@
   AXIS SIGNS ARE PROVISIONAL: lengths, parallelism and anchors are
   caliper-measured; the world-direction of each joint's positive sense
-  still needs the first powered RViz-vs-reality comparison (v0.2 session,
-  one small commanded angle per joint). A wrong sense is a one-line flip
-  here plus the same flip in the mirror. Do not "fix" signs from the
-  armchair; fix them from the bench.
+  is checked joint by joint by soma_sign_check (v0.2). Two findings, two
+  different fixes. METAL moving opposite to the hug convention is a
+  driver fix: mirror the joint's SERVO_MAP row and sync its limits here
+  (macro defaults for the right arm, the bench call for the left). It is
+  never an axis flip: every planar <axis> below uses ${side}, so a flip
+  changes both arms. RViz drawing a joint the other way while the metal
+  is right is the case for an <axis> flip, and a flip only one arm needs
+  takes a per-side parameter, not an edit of the shared line. Do not
+  "fix" signs from the armchair; fix them from the bench.
   Visuals are honest bounding boxes; pretty geometry arrives with the
   CAD-to-URDF pipeline (task #30). Roughly 0.7 kg per hanging arm (the

Commit message: Model fixed against the metal: wrist roll and finger axes, pinned by an FK test
The sign check passed 12 of 12 on the metal on 2026-10-12, so the driver
was right everywhere. The model was not: seen from above, a negative
wrist roll turns the gripper inward on the metal (counterclockwise on
the right arm, clockwise on the left, as Andres saw it), and the URDF
drew both the other way. The URDF also drew a positive finger command
as the two fingers closing and crossing, while the metal opens.

soma_arm.xacro: the wrist roll axis goes from ${side} to ${-side} and
both finger axes from 0 1 0 to 0 -1 0. Both arms disagreed the same
way, so the shared lines are the right place. The driver, the joint
limits and the reach map do not change (the map only uses the four
planar joints, whose drawing was already right).

test_model_directions.py runs a generic forward kinematics over the
bench URDF and pins, per arm: a negative yaw, shoulder, elbow or wrist
pitch swings the tool forward; a negative roll turns the gripper
inward; a positive finger command opens without crossing. On the URDF
produced by the Jetson's container before this change, 4 of its 12
cases failed (the rolls and the fingers); with the three lines flipped,
12 of 12 pass. It needs xacro (the unit job installs it) or a URDF named
by SOMA_URDF.

sign_check.py quotes the current axis lines in its model fixes; they
follow the change, and a new test checks that every quoted line is in
the xacro. Tests edited on purpose: the two assertions on those quoted
lines, because the model they describe changed.

Also: the left arm's report (6 of 6 ok) and the log entry completed.

Co-Authored-By: Claude Opus 5.5 <noreply@anthropic.com>

File: soma_description/urdf/soma_arm.xacro (robot description, xacro)
@@ -27,8 +27,9 @@
   mirror-symmetric between arms by definition, so the left arm uses
   side=1 and the right arm side=-1 on every revolute axis.
-  AXIS SIGNS ARE PROVISIONAL: lengths, parallelism and anchors are
-  caliper-measured; the world-direction of each joint's positive sense
-  is checked joint by joint by soma_sign_check (v0.2). Two findings, two
-  different fixes. METAL moving opposite to the hug convention is a
+  AXIS SIGNS, VERIFIED 2026-10-12: the sign check passed 12 of 12 on the
+  metal, and soma_driver/test/test_model_directions.py runs the FK of
+  this model to pin that it draws every joint the way the metal moves
+  (the wrist roll and the fingers were drawn backwards until that day).
+  For any future joint or servo, two findings, two different fixes. METAL moving opposite to the hug convention is a
   driver fix: mirror the joint's SERVO_MAP row and sync its limits here
   (macro defaults for the right arm, the bench call for the left). It is
@@ -192,5 +193,8 @@
       <child link="${prefix}gripper_base_link"/>
       <origin xyz="${wrist_len} 0 0"/>
-      <axis xyz="${side} 0 0"/>
+      <!-- ${-side}, not ${side}: a negative roll turns the gripper inward,
+           CCW seen from above on the right arm, CW on the left (seen on the
+           metal 2026-10-12; test_model_directions.py pins it). -->
+      <axis xyz="${-side} 0 0"/>
       <limit lower="${wrist_roll_lower}" upper="${wrist_roll_upper}" effort="${effort_nm}" velocity="${vel_rads}"/>
     </joint>
@@ -212,5 +216,7 @@
       <child link="${prefix}finger_l_link"/>
       <origin xyz="${gripper_base_h} 0 ${finger_sep/2}"/>
-      <axis xyz="0 1 0"/>
+      <!-- 0 -1 0: a positive command OPENS (the tips move apart). With 0 1 0
+           the model drew 1.0 as two crossed fingers (fixed 2026-10-12). -->
+      <axis xyz="0 -1 0"/>
       <limit lower="0.0" upper="1.0" effort="${effort_nm}" velocity="${vel_rads}"/>
     </joint>
@@ -231,5 +237,5 @@
       <child link="${prefix}finger_r_link"/>
       <origin xyz="${gripper_base_h} 0 ${-finger_sep/2}"/>
-      <axis xyz="0 1 0"/>
+      <axis xyz="0 -1 0"/>
       <limit lower="-1.0" upper="0.0" effort="${effort_nm}" velocity="${vel_rads}"/>
       <mimic joint="${prefix}finger_l_joint" multiplier="-1.0"/>

Commit message: Dimensions re-measured with a caliper; the IK works in the measured lane
The arm chain moved by about 1 mm a link. The tool is now one direct
reading (150.0 closed, about 100 open), and the IK uses it rather than
the sum of its parts. The lane is the measured 81 mm, half the 162
between the closed tips: the model gains a plane offset along the
parallel axes (a DH d) so its chain works there too. mount_h is left as
it was until a disc-to-tip reading settles a 42 mm disagreement.

Co-Authored-By: Claude Opus 5.5 <noreply@anthropic.com>

File: soma_description/urdf/soma_arm.xacro (robot description, xacro)
@@ -44,15 +44,18 @@
 -->
 <robot xmlns:xacro="http://www.ros.org/wiki/xacro">
-  <!-- ============ dimensions, MEASURED 2026-08-05 ============
+  <!-- ============ dimensions, MEASURED 2026-08-05, re-measured 2026-10-27 ============
        Every literal here has a provenance row in config/dimensions.yaml;
        test_dimensions_sync.py keeps the two in agreement. -->
   <xacro:property name="disc_r"         value="0.02455"/> <!-- slew disc, the one that rotates -->
-  <xacro:property name="disc_h"         value="0.0074"/>  <!-- disc protrusion from its box -->
-  <xacro:property name="clavicle_len"   value="0.033"/>   <!-- disc center to shoulder axis -->
-  <xacro:property name="upper_len"      value="0.0793"/>  <!-- shoulder to elbow -->
-  <xacro:property name="fore_len"       value="0.075"/>   <!-- elbow to wrist pitch -->
-  <xacro:property name="wrist_len"      value="0.0664"/>  <!-- wrist pitch to gripper mount face -->
-  <xacro:property name="gripper_base_h" value="0.0179"/>  <!-- mount face to finger gear axes -->
-  <xacro:property name="finger_len"     value="0.0657"/>  <!-- gear axis to fingertip -->
+  <xacro:property name="disc_h"         value="0.0097"/>  <!-- disc protrusion from its box -->
+  <xacro:property name="clavicle_len"   value="0.0327"/>   <!-- disc center to shoulder axis -->
+  <xacro:property name="upper_len"      value="0.0800"/>  <!-- shoulder to elbow -->
+  <xacro:property name="fore_len"       value="0.0760"/>   <!-- elbow to wrist pitch -->
+  <xacro:property name="wrist_len"      value="0.0663"/>  <!-- wrist pitch to gripper mount face -->
+  <xacro:property name="gripper_base_h" value="0.0178"/>  <!-- mount face to finger gear axes -->
+  <xacro:property name="finger_len"     value="0.0650"/>  <!-- gear axis to fingertip -->
+  <xacro:property name="tool_closed_len" value="0.150"/>  <!-- wrist pitch axis to fingertip, closed, one reading (the IK tool) -->
+  <xacro:property name="tool_open_len"  value="0.100"/>   <!-- wrist pitch axis to the farthest point, fully open -->
+  <xacro:property name="plane_offset"   value="0.02725"/> <!-- working plane outboard of the disc face: a DH d -->
   <xacro:property name="finger_sep"     value="0.0257"/>  <!-- between the two gear axes -->
   <xacro:property name="plate_w"        value="0.0319"/>  <!-- link plate width -->
@@ -132,5 +135,7 @@
       <parent link="${prefix}turntable_link"/>
       <child link="${prefix}upper_arm_link"/>
-      <origin xyz="${clavicle_len} 0 ${disc_h}"/>
+      <!-- z: the disc face plus the plane offset, so the planar chain and
+           the fingertip work in the measured lane (2026-10-27). -->
+      <origin xyz="${clavicle_len} 0 ${disc_h + plane_offset}"/>
       <axis xyz="0 0 ${side}"/>
       <limit lower="${shoulder_lower}" upper="${shoulder_upper}" effort="${effort_nm}" velocity="${vel_rads}"/>

File: soma_description/urdf/soma_bench.urdf.xacro (robot description, xacro)
@@ -28,6 +28,7 @@
        Provenance for every literal: config/dimensions.yaml, bench section. -->
   <xacro:property name="mount_lx"     value="0.0811"/>  <!-- central box front-back -->
-  <xacro:property name="mount_ly"     value="0.1098"/>  <!-- disc seat to disc seat -->
+  <xacro:property name="mount_ly"     value="0.0881"/>  <!-- disc seat to disc seat -->
   <xacro:property name="mount_lz"     value="0.0856"/>  <!-- central box top-bottom -->
+  <xacro:property name="tip_lane_y"   value="0.081"/>   <!-- closed tip lane, half the 162 mm between tips -->
   <xacro:property name="mount_h"      value="0.343"/>   <!-- disc axis over the plate -->
   <xacro:property name="plate_lx"     value="0.220"/>

Commit message: The clavicle rises: a DH theta offset closes the 45 mm gap
The hanging right arm measured 295 mm disc to tip against 338.7 in the
model. From the side, the OAK showed the shoulder axis 15.6 mm above the
disc axis, behind it, and the rest of the arm hanging straight with the
caliper lengths. The clavicle leaves the disc at 118.5 deg from straight
down; the shoulder's zero takes it back out. clavicle_angle goes into
dimensions.yaml, the xacro and the IK; mount_h is re-measured at 327.2.
The FK now predicts the hanging tip 36.8 mm over the plate against 38
measured, pinned by a test.

Co-Authored-By: Claude Opus 5.5 <noreply@anthropic.com>

File: soma_description/urdf/soma_arm.xacro (robot description, xacro)
@@ -55,4 +55,5 @@
   <xacro:property name="gripper_base_h" value="0.0178"/>  <!-- mount face to finger gear axes -->
   <xacro:property name="finger_len"     value="0.0650"/>  <!-- gear axis to fingertip -->
+  <xacro:property name="clavicle_angle" value="2.068"/>   <!-- rad: clavicle direction at the hanging zero, from down, backward (DH theta offset) -->
   <xacro:property name="tool_closed_len" value="0.150"/>  <!-- wrist pitch axis to fingertip, closed, one reading (the IK tool) -->
   <xacro:property name="tool_open_len"  value="0.100"/>   <!-- wrist pitch axis to the farthest point, fully open -->
@@ -137,5 +138,10 @@
       <!-- z: the disc face plus the plane offset, so the planar chain and
            the fingertip work in the measured lane (2026-10-27). -->
-      <origin xyz="${clavicle_len} 0 ${disc_h + plane_offset}"/>
+      <!-- The clavicle leaves the disc at clavicle_angle (measured 2026-10-27:
+           the shoulder axis sits 15.6 mm above the disc axis, behind it). The
+           frame turns back by the same angle, so the upper arm still hangs
+           straight down at a zero shoulder. -->
+      <origin xyz="${clavicle_len*cos(clavicle_angle)} ${side*clavicle_len*sin(clavicle_angle)} ${disc_h + plane_offset}"
+              rpy="0 0 ${-side*clavicle_angle}"/>
       <axis xyz="0 0 ${side}"/>
       <limit lower="${shoulder_lower}" upper="${shoulder_upper}" effort="${effort_nm}" velocity="${vel_rads}"/>

File: soma_description/urdf/soma_bench.urdf.xacro (robot description, xacro)
@@ -31,5 +31,5 @@
   <xacro:property name="mount_lz"     value="0.0856"/>  <!-- central box top-bottom -->
   <xacro:property name="tip_lane_y"   value="0.081"/>   <!-- closed tip lane, half the 162 mm between tips -->
-  <xacro:property name="mount_h"      value="0.343"/>   <!-- disc axis over the plate -->
+  <xacro:property name="mount_h"      value="0.3272"/>   <!-- disc axis over the plate -->
   <xacro:property name="plate_lx"     value="0.220"/>
   <xacro:property name="plate_ly"     value="0.280"/>

Commit message: xacro: the clavicle offset moves the shoulder origin only, not its frame
Turning the shoulder frame back by the clavicle angle twisted the whole
arm in the URDF (test_model_directions caught the tip moving backward on
a forward command). The frame keeps the turntable's orientation; only
the origin moves.

Co-Authored-By: Claude Opus 5.5 <noreply@anthropic.com>

File: soma_description/urdf/soma_arm.xacro (robot description, xacro)
@@ -139,9 +139,9 @@
            the fingertip work in the measured lane (2026-10-27). -->
       <!-- The clavicle leaves the disc at clavicle_angle (measured 2026-10-27:
-           the shoulder axis sits 15.6 mm above the disc axis, behind it). The
-           frame turns back by the same angle, so the upper arm still hangs
-           straight down at a zero shoulder. -->
-      <origin xyz="${clavicle_len*cos(clavicle_angle)} ${side*clavicle_len*sin(clavicle_angle)} ${disc_h + plane_offset}"
-              rpy="0 0 ${-side*clavicle_angle}"/>
+           the shoulder axis sits 15.6 mm above the disc axis, behind it).
+           Only the origin moves: the frame keeps the turntable's
+           orientation, so the upper arm still hangs straight down at a
+           zero shoulder. -->
+      <origin xyz="${clavicle_len*cos(clavicle_angle)} ${side*clavicle_len*sin(clavicle_angle)} ${disc_h + plane_offset}"/>
       <axis xyz="0 0 ${side}"/>
       <limit lower="${shoulder_lower}" upper="${shoulder_upper}" effort="${effort_nm}" velocity="${vel_rads}"/>
